File: high_current_v1/rev-/fet_switch.kicad_pcb (KiCad board)
At the start: 2 copper layers, 38.1 x 31.8 mm, 17 parts, among them Q1 FQP27P06, Q2 MMBTA06LT1G

Commit message: fixed silkscreen...resistor identifiers changed to match W6PQL schematic and table.
Parts:
- renumbered R2 to R1, R5 to R2, R7 to R3, R1 to R4, R3 to R5, R4 to R6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
