File: high_current_v1/rev-/fet_switch.sch (KiCad schematic (older format))
At the start: 17 parts, among them Q1 FQP27P06, Q2 MMBTA06LT1G

Commit message: fixed silkscreen...resistor identifiers changed to match W6PQL schematic and table.
Parts:
- renumbered R2 to R1, R5 to R2, R7 to R3, R1 to R4, R3 to R5, R4 to R6, R6 to R7
Changed lines of the file:
@@
 $EndComp
 $Comp
-L Device:R_US R2
+L Device:R_US R1
 U 1 1 5ED33A03
 P 4250 3800
-F 0 "R2" H 4318 3846 50  0000 L CNN
+F 0 "R1" H 4318 3846 50  0000 L CNN
 F 1 "1k" H 4318 3755 50  0000 L CNN
 F 2 "digikey-footprints:0805" V 4290 3790 50  0001 C CNN
@@
 $EndComp
 $Comp
-L Device:R_US R5
+L Device:R_US R2
 U 1 1 5ED351C0
 P 4250 4200
-F 0 "R5" H 4318 4246 50  0000 L CNN
+F 0 "R2" H 4318 4246 50  0000 L CNN
 F 1 "6k" H 4318 4155 50  0000 L CNN
 F 2 "digikey-footprints:0805" V 4290 4190 50  0001 C CNN
@@
 $EndComp
 $Comp
-L Device:R_US R7
+L Device:R_US R3
 U 1 1 5ED35789
 P 4250 4600
-F 0 "R7" H 4318 4646 50  0000 L CNN
+F 0 "R3" H 4318 4646 50  0000 L CNN
 F 1 "2k" H 4318 4555 50  0000 L CNN
 F 2 "digikey-footprints:0805" V 4290 4590 50  0001 C CNN
@@
 $EndComp
 $Comp
-L Device:R_US R6
+L Device:R_US R7
 U 1 1 5ED35D74
 P 3500 4600
-F 0 "R6" H 3568 4646 50  0000 L CNN
+F 0 "R7" H 3568 4646 50  0000 L CNN
 F 1 "2.5k" H 3568 4555 50  0000 L CNN
 F 2 "digikey-footprints:0805" V 3540 4590 50  0001 C CNN
@@
 $EndComp
 $Comp
-L Device:R_US R4
+L Device:R_US R6
 U 1 1 5ED36A92
 P 3500 4200
-F 0 "R4" H 3568 4246 50  0000 L CNN
+F 0 "R6" H 3568 4246 50  0000 L CNN
 F 1 "8k" H 3568 4155 50  0000 L CNN
 F 2 "digikey-footprints:0805" V 3540 4190 50  0001 C CNN
@@
 $EndComp
 $Comp
-L Device:R_US R3
+L Device:R_US R5
 U 1 1 5ED3BCD8
 P 5000 4050
-F 0 "R3" H 5068 4096 50  0000 L CNN
+F 0 "R5" H 5068 4096 50  0000 L CNN
 F 1 "500" H 5068 4005 50  0000 L CNN
 F 2 "digikey-footprints:0805" V 5040 4040 50  0001 C CNN
@@
 $EndComp
 $Comp
-L Device:R_US R1
+L Device:R_US R4
 U 1 1 5ED3C6E3
 P 4600 3750
-F 0 "R1" H 4668 3796 50  0000 L CNN
+F 0 "R4" H 4668 3796 50  0000 L CNN
 F 1 "10k" H 4668 3705 50  0000 L CNN
 F 2 "digikey-footprints:0805" V 4640 3740 50  0001 C CNN
